File: My Keyboard.kicad_pcb (KiCad board)
At the start: 2 copper layers, 383.8 x 135.4 mm, 293 parts, among them J1 OLED_128x64, U1 Raspberry_Pi_Pico

Commit message: some changes
Routing:
- net +5V: track 0.00 -> 2382.5 mm, vias 0 -> 2
- net GND: track 0.00 -> 2295.0 mm
- net Column 4: track 684.2 -> 0.00 mm, vias 20 -> 0
- net Column 3: track 648.8 -> 0.00 mm, vias 27 -> 0
- net Column 0: track 632.8 -> 0.00 mm, vias 12 -> 0
- net Column 2: track 612.6 -> 0.00 mm, vias 14 -> 0
- net Column 7: track 588.4 -> 0.00 mm, vias 36 -> 0
- net Column 9: track 550.3 -> 0.00 mm, vias 40 -> 0
- net Column 8: track 544.2 -> 0.00 mm, vias 42 -> 0
- net Column 1: track 531.8 -> 0.00 mm, vias 12 -> 0
- net Column 10: track 520.2 -> 0.00 mm, vias 42 -> 0
- net Column 5: track 505.9 -> 0.00 mm, vias 34 -> 0
- net Column 6: track 505.7 -> 0.00 mm, vias 40 -> 0
- net Column 11: track 504.0 -> 0.00 mm, vias 54 -> 0
- net Row 6: track 454.5 -> 0.00 mm
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
Commit message: final touches.
Parts:
- added U2: PCF8574P, Package_DIP:DIP-16_W7.62mm, F.Cu at (31.3, 26.9)
- moved D130 0.92 mm to (386.6, 71.3)
- moved D192 0.33 mm to (338.1, 147.3)
Connections:
- net +5V renamed +3.3V
- D100 pad 1: Row 6 -> Row 5
- D101 pad 1: Row 6 -> Row 5
- D102 pad 1: Row 6 -> Row 5
- D15 pad 1: Row 1 -> Row 0
- D29 pad 1: Row 2 -> Row 1
- D30 pad 1: Row 2 -> Row 1
- D31 pad 1: Row 2 -> Row 1
- D32 pad 1: Row 2 -> Row 1
- D33 pad 1: Row 2 -> Row 1
- D43 pad 1: Row 3 -> Row 2
- D44 pad 1: Row 3 -> Row 2
- D45 pad 1: Row 3 -> Row 2
- D46 pad 1: Row 3 -> Row 2
- D47 pad 1: Row 3 -> Row 2
- D49 pad 1: Row 3 -> Row 2
- D50 pad 1: Row 3 -> Row 2
- D51 pad 1: Row 3 -> Row 2
- D53 pad 1: Row 3 -> Row 2
- D61 pad 1: Row 4 -> Row 3
- D62 pad 1: Row 4 -> Row 3
- D63 pad 1: Row 4 -> Row 3
- D65 pad 1: Row 4 -> Row 3
- D66 pad 1: Row 4 -> Row 3
- D67 pad 1: Row 4 -> Row 3
- D68 pad 1: Row 4 -> Row 3
- D69 pad 1: Row 4 -> Row 3
- D70 pad 1: Row 4 -> Row 3
- D71 pad 1: Row 4 -> Row 3
- D72 pad 1: Row 4 -> Row 3
- D76 pad 1: Row 5 -> Row 4
- D77 pad 1: Row 5 -> Row 4
- D78 pad 1: Row 5 -> Row 4
- D79 pad 1: Row 5 -> Row 4
- D80 pad 1: Row 5 -> Row 4
- D81 pad 1: Row 5 -> Row 4
- D82 pad 1: Row 5 -> Row 4
- D83 pad 1: Row 5 -> Row 4
- D84 pad 1: Row 5 -> Row 4
- D85 pad 1: Row 5 -> Row 4
- D86 pad 1: Row 5 -> Row 4
- D87 pad 1: Row 5 -> Row 4
- D88 pad 1: Row 5 -> Row 4
- D89 pad 1: Row 5 -> Row 4
- D90 pad 1: Row 6 -> Row 4
- D91 pad 1: Row 6 -> Row 5
- D92 pad 1: Row 6 -> Row 5
- D93 pad 1: Row 6 -> Row 5
- D94 pad 1: Row 6 -> Row 5
- D95 pad 1: Row 6 -> Row 5
- D96 pad 1: Row 6 -> Row 5
- D97 pad 1: Row 6 -> Row 5
- D98 pad 1: Row 6 -> Row 5
- D99 pad 1: Row 6 -> Row 5
- S15 pad 1: Column 0 -> Column 14
- S16 pad 1: Column 1 -> Column 0
- S17 pad 1: Column 2 -> Column 1
- S18 pad 1: Column 3 -> Column 2
- S19 pad 1: Column 4 -> Column 3
- S20 pad 1: Column 5 -> Column 4
- S21 pad 1: Column 6 -> Column 5
- S22 pad 1: Column 7 -> Column 6
- S23 pad 1: Column 8 -> Column 7
- S24 pad 1: Column 9 -> Column 8
- S25 pad 1: Column 10 -> Column 9
- S26 pad 1: Column 11 -> Column 10
- S27 pad 1: Column 12 -> Column 11
- S28 pad 1: Column 13 -> Column 12
- S29 pad 1: Column 0 -> Column 13
- S30 pad 1: Column 1 -> Column 14
- S31 pad 1: Column 2 -> Column 15
- S32 pad 1: Column 3 -> Column 16
- S33 pad 1: Column 4 -> Column 17
- S34 pad 1: Column 5 -> Column 0
- S35 pad 1: Column 6 -> Column 1
- S36 pad 1: Column 7 -> Column 2
- S37 pad 1: Column 8 -> Column 3
- S38 pad 1: Column 9 -> Column 4
- S39 pad 1: Column 10 -> Column 5
- S40 pad 1: Column 11 -> Column 6
- S41 pad 1: Column 12 -> Column 7
- S42 pad 1: Column 13 -> Column 8
- S43 pad 1: Column 0 -> Column 9
- S44 pad 1: Column 1 -> Column 10
- S45 pad 1: Column 2 -> unconnected-(S45-Pad1)
- S46 pad 1: Column 3 -> Column 12
- S47 pad 1: Column 4 -> Column 13
- S48 pad 1: Column 5 -> Column 14
- S49 pad 1: Column 6 -> Column 15
- S50 pad 1: Column 7 -> Column 16
- S51 pad 1: Column 8 -> Column 17
- S52 pad 1: Column 9 -> Column 0
- S53 pad 1: Column 10 -> Column 1
- S54 pad 1: Column 11 -> Column 2
- S55 pad 1: Column 12 -> Column 3
- S56 pad 1: Column 13 -> Column 4
- S57 pad 1: Column 0 -> Column 5
- S58 pad 1: Column 1 -> Column 6
- S59 pad 1: Column 2 -> Column 7
- S60 pad 1: Column 3 -> Column 8
- S61 pad 1: Column 4 -> Column 9
- S62 pad 1: Column 5 -> Column 10
- S63 pad 1: Column 6 -> unconnected-(S63-Pad1)
- S64 pad 1: Column 7 -> Column 13
- S65 pad 1: Column 8 -> Column 14
- S66 pad 1: Column 9 -> Column 15
- S67 pad 1: Column 10 -> Column 16
- S68 pad 1: Column 11 -> Column 0
- S69 pad 1: Column 12 -> Column 1
- S70 pad 1: Column 13 -> Column 2
- S71 pad 1: Column 0 -> Column 3
- S72 pad 1: Column 1 -> Column 4
- S73 pad 1: Column 2 -> Column 5
- S74 pad 1: Column 3 -> Column 6
- S75 pad 1: Column 4 -> Column 7
- S76 pad 1: Column 5 -> Column 8
- S77 pad 1: Column 6 -> Column 9
- S78 pad 1: Column 7 -> Column 10
- S79 pad 1: Column 8 -> unconnected-(S79-Pad1)
- S80 pad 1: Column 9 -> Column 12
- S81 pad 1: Column 10 -> Column 13
- S82 pad 1: Column 11 -> unconnected-(S82-Pad1)
- S83 pad 1: Column 12 -> Column 15
- S84 pad 1: Column 13 -> Column 16
- S85 pad 1: Column 0 -> Column 17
- S86 pad 1: Column 1 -> Column 0
- S87 pad 1: Column 2 -> Column 1
- S88 pad 1: Column 3 -> Column 2
- S89 pad 1: Column 4 -> Column 3
- S90 pad 1: Column 5 -> Column 4
- S91 pad 1: Column 6 -> Column 9
- S92 pad 1: Column 7 -> Column 10
- S93 pad 1: Column 8 -> unconnected-(S93-Pad1)
- S94 pad 1: Column 9 -> Column 12
- S95 pad 1: Column 10 -> Column 13
- S96 pad 1: Column 11 -> unconnected-(S96-Pad1)
- S97 pad 1: Column 12 -> Column 16
- U1 pad 17: Column 13 -> SCL
- U1 pad 26: Row 6 -> unconnected-(U1-GPIO20-Pad26)
- U1 pad 29: unconnected-(U1-GPIO22-Pad29) -> SDA
- U1 pad 31: SDA -> unconnected-(U1-GPIO26_ADC0-Pad31)
- U1 pad 32: SCL -> unconnected-(U1-GPIO27_ADC1-Pad32)
Routing:
- net Column 13: track 0.00 -> 727.9 mm, vias 0 -> 12
- net Column 14: track 0.00 -> 577.2 mm, vias 0 -> 7
- net Column 16: track 0.00 -> 557.7 mm
- net Column 9: track 0.00 -> 521.9 mm, vias 0 -> 8
- net Column 15: track 0.00 -> 517.9 mm
- net Column 0: track 0.00 -> 480.5 mm
- net Column 1: track 0.00 -> 466.8 mm
- net Column 17: track 0.00 -> 465.7 mm
- net Column 2: track 0.00 -> 454.5 mm
- net Row 5: track 0.00 -> 442.9 mm, vias 0 -> 20
- net Column 7: track 0.00 -> 442.7 mm, vias 0 -> 4
- net Column 4: track 0.00 -> 434.6 mm, vias 0 -> 2
- net Column 3: track 0.00 -> 430.1 mm, vias 0 -> 2
- net Row 4: track 0.00 -> 422.8 mm, vias 0 -> 20
- net Row 2: track 0.00 -> 388.5 mm, vias 0 -> 6
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Other:
- board size 383.8 x 135.4 mm -> 376.7 x 135.5 mm
