File: My Keyboard.kicad_sch (KiCad schematic)
At the start: 293 parts, among them J1 OLED_128x64, U1 Raspberry_Pi_Pico

Commit message: final touches.
Parts:
- added U2: PCF8574P, Package_DIP:DIP-16_W7.62mm, symbol Interface_Expansion:PCF8574P
Connections:
- net Column 0: now also S16.1, S34.1, S52.1, S68.1, S86.1; no longer S15.1, S29.1, S43.1, S57.1, S71.1, S85.1
- net Column 1: now also S17.1, S35.1, S53.1, S69.1, S87.1; no longer S16.1, S30.1, S44.1, S58.1, S72.1, S86.1
- net Column 10: now also S26.1, S44.1, S62.1, S78.1, S92.1; no longer S25.1, S39.1, S53.1, S67.1, S81.1, S95.1
- net Column 11: now also S27.1; no longer S26.1, S40.1, S54.1, S68.1, S82.1, S96.1
- net Column 12: now also S28.1, S46.1, S80.1, S94.1; no longer S27.1, S41.1, S55.1, S69.1, S83.1, S97.1
- net Column 13: now also S29.1, S47.1, S64.1, S81.1, S95.1, U2.4 (P0); no longer S28.1, S42.1, S56.1, S70.1, S84.1, U1.17 (GPIO13)
- net Column 2: now also S18.1, S36.1, S54.1, S70.1, S88.1; no longer S17.1, S31.1, S45.1, S59.1, S73.1, S87.1
- net Column 3: now also S19.1, S37.1, S55.1, S71.1, S89.1; no longer S18.1, S32.1, S46.1, S60.1, S74.1, S88.1
- net Column 4: now also S20.1, S38.1, S56.1, S72.1, S90.1; no longer S19.1, S33.1, S47.1, S61.1, S75.1, S89.1
- net Column 5: now also S21.1, S39.1, S57.1, S73.1; no longer S20.1, S34.1, S48.1, S62.1, S76.1, S90.1
- net Column 6: now also S22.1, S40.1, S58.1, S74.1; no longer S21.1, S35.1, S49.1, S63.1, S77.1, S91.1
- net Column 7: now also S23.1, S41.1, S59.1, S75.1; no longer S22.1, S36.1, S50.1, S64.1, S78.1, S92.1
- net Column 8: now also S24.1, S42.1, S60.1, S76.1; no longer S23.1, S37.1, S51.1, S65.1, S79.1, S93.1
- net Column 9: now also S25.1, S43.1, S61.1, S77.1, S91.1; no longer S24.1, S38.1, S52.1, S66.1, S80.1, S94.1
- net GND: now also U2.1 (A0), U2.2 (A1), U2.3 (A2), U2.8 (GND)
- net Row 0: now also D15.1 (K)
- net Row 1: now also D29.1 (K), D30.1 (K), D31.1 (K), D32.1 (K), D33.1 (K); no longer D15.1 (K)
- net Row 2: now also D43.1 (K), D44.1 (K), D45.1 (K), D46.1 (K), D47.1 (K), D49.1 (K), D50.1 (K), D51.1 (K), D53.1 (K); no longer D29.1 (K), D30.1 (K), D31.1 (K), D32.1 (K), D33.1 (K)
- net Row 3: now also D61.1 (K), D62.1 (K), D63.1 (K), D65.1 (K), D66.1 (K), D67.1 (K), D68.1 (K), D69.1 (K), D70.1 (K), D71.1 (K), D72.1 (K); no longer D43.1 (K), D44.1 (K), D45.1 (K), D46.1 (K), D47.1 (K), D49.1 (K), D50.1 (K), D51.1 (K), D53.1 (K)
- net Row 4: now also D76.1 (K), D77.1 (K), D78.1 (K), D79.1 (K), D80.1 (K), D81.1 (K), D82.1 (K), D83.1 (K), D84.1 (K), D85.1 (K), D86.1 (K), D87.1 (K), D88.1 (K), D89.1 (K), D90.1 (K); no longer D61.1 (K), D62.1 (K), D63.1 (K), D65.1 (K), D66.1 (K), D67.1 (K), D68.1 (K), D69.1 (K), D70.1 (K), D71.1 (K), D72.1 (K)
- net Row 5: now also D100.1 (K), D101.1 (K), D102.1 (K), D91.1 (K), D92.1 (K), D93.1 (K), D94.1 (K), D95.1 (K), D96.1 (K), D97.1 (K), D98.1 (K), D99.1 (K); no longer D76.1 (K), D77.1 (K), D78.1 (K), D79.1 (K), D80.1 (K), D81.1 (K), D82.1 (K), D83.1 (K), D84.1 (K), D85.1 (K), D86.1 (K), D87.1 (K), D88.1 (K), D89.1 (K)
- net SCL: now also U1.17 (GPIO13), U2.14 (SCL); no longer U1.32 (GPIO27_ADC1)
- net SDA: now also U1.29 (GPIO22), U2.15 (SDA); no longer U1.31 (GPIO26_ADC0)
- net +5V renamed +3.3V
- net +3.3V: now also U2.16 (VDD)
- removed net Row 6: D100.1 (K), D101.1 (K), D102.1 (K), D90.1 (K), D91.1 (K), D92.1 (K), D93.1 (K), D94.1 (K), D95.1 (K), D96.1 (K), D97.1 (K), D98.1 (K), D99.1 (K), U1.26 (GPIO20)
- new net Column 14: S15.1, S30.1, S48.1, S65.1, U2.5 (P1)
- new net Column 15: S31.1, S49.1, S66.1, S83.1, U2.6 (P2)
- new net Column 16: S32.1, S50.1, S67.1, S84.1, S97.1, U2.7 (P3)
- new net Column 17: S33.1, S51.1, S85.1, U2.9 (P4)
Other:
- moved on the sheet: D1, D10, D100, D101, D102, D11, D12, D13, D14, D15, D16, D17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
