File: Kicad/My Keyboard.kicad_pcb (KiCad board)
At the start: 2 copper layers, 290.9 x 128.4 mm, 185 parts, among them J1 OLED_128x64, U1 Raspberry_Pi_Pico

Commit message: .
Parts:
- S1, S10, S11, S12, S13, S14, S15, S16, S17, S18, S19, S2, S20, S21, S22, S23, S24, S25, S26, S27, S28, S29, S3, S30, S31, S32, S33, S34, S35, S36, S37, S38, S39, S4, S40, S41, S42, S43, S44, S45, S46, S47, S48, S49, S5, S50, S51, S52, S53, S54, S55, S56, S57, S58, S59, S6, S60, S61, S7, S8, S9: footprint ScottoKeebs_MX:MX_PCB_1.00u -> Button_Switch_Keyboard:SW_Cherry_MX_1.00u_PCB
- moved S13 5.68 mm to (269.2, 33.0)
- moved S14 5.68 mm to (297.8, 33.0)
- moved S24 5.68 mm to (221.6, 52.1)
- moved S34 5.68 mm to (150.2, 71.1)
- moved S39 5.68 mm to (245.4, 71.1)
- moved S40 5.68 mm to (264.5, 71.1)
- moved S49 5.68 mm to (197.8, 90.2)
- moved S57 5.68 mm to (162.1, 109.2)
- moved S58 5.68 mm to (233.5, 109.2)
- moved S59 5.68 mm to (257.3, 109.2)
- moved S60 5.68 mm to (281.1, 109.2)
- moved S61 5.68 mm to (305.0, 109.2)
- moved S8 5.68 mm to (174.0, 33.0)
- moved S15 5.68 mm to (45.4, 52.1)
- moved S16 5.68 mm to (69.2, 52.1)
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Routing:
- net GND: track 1497.4 -> 0.00 mm
- net +5V: track 1484.1 -> 0.00 mm, vias 8 -> 0
- net Column 1: track 477.3 -> 0.00 mm, vias 8 -> 0
- net Column 0: track 378.2 -> 0.00 mm, vias 4 -> 0
- net Row 4: track 375.0 -> 0.00 mm, vias 8 -> 0
- net Column 2: track 371.6 -> 0.00 mm, vias 12 -> 0
- net Column 3: track 364.2 -> 0.00 mm, vias 14 -> 0
- net Row 3: track 342.1 -> 0.00 mm, vias 6 -> 0
- net Row 1: track 329.8 -> 0.00 mm, vias 2 -> 0
- net Row 2: track 325.7 -> 0.00 mm, vias 4 -> 0
- net Column 12: track 315.6 -> 0.00 mm, vias 8 -> 0
- net Column 4: track 307.7 -> 0.00 mm, vias 12 -> 0
- net Row 0: track 306.7 -> 0.00 mm
- net Column 5: track 261.5 -> 0.00 mm, vias 12 -> 0
- net Column 6: track 230.4 -> 0.00 mm, vias 16 -> 0
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