File: Kicad/My Keyboard.kicad_sch (KiCad schematic)
At the start: 185 parts, among them J1 OLED_128x64, U1 Raspberry_Pi_Pico

Commit message: .
Parts:
- S1, S10, S11, S12, S13, S14, S15, S16, S17, S18, S19, S2, S20, S21, S22, S23, S24, S25, S26, S27, S28, S29, S3, S30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: footprint ScottoKeebs_MX:MX_PCB_1.00u -> Button_Switch_Keyboard:SW_Cherry_MX_1.00u_PCB
Connections:
- net +3.3V: now also U1.36 (3V3); no longer U1.40 (VBUS)
- no-connect marks 0 -> 19
Other:
- moved on the sheet: D1, D10, D100, D101, D102, D103, D104, D105, D106, D107, D108, D109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
